File: hw/sch_pcb/DIG4SWHI01.kicad_sch (KiCad schematic)
At the start: 51 parts, among them J1 CONN1_1, J10 JUMP_2x1, J11 JUMP_2x1, J12 CONN1_1, J13 CONN1_1, J14 CONN1_1, J15 CONN1_1, J16 CONN1_1, J17 CONN1_1, J18 CONN1_1, J19 CONN1_1, J2 CONN1_1, J20 JUMP_2x1, J3 JUMP_2x1, J4 JUMP_2x1, J5 JUMP_2x1, J6 JUMP_2x1, J7 JUMP_2x1, J8 JUMP_2x1, J9 JUMP_2x1, M1 HOLE, M2 HOLE, M3 HOLE, M4 HOLE, U1 VNQ7050AJ

Commit message: Attempt to resolve action fail.
Other:
- title: NAME -> DIG4SWHI01
